File: temp_sensor.kicad_sch (KiCad schematic)
At the start: 26 parts, among them J2 Conn_01x06, J3 Conn_01x08, J4 Conn_01x08, SW1 Boot, SW2 Reset, U1 HDC3020DEFR, U2 ESP-12F, U3 TPS613221ADBVR, U4 TLV74033PDBVR

Commit message: Added cap at reset and screw hole
Parts:
- added C3: 10nF, Capacitor_SMD:C_0603_1608Metric_Pad1.08x0.95mm_HandSolder, symbol Device:C
Connections:
- net GNDREF: now also C3.2
- net wake: now also C3.1
Changed lines of the file:
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@@
 	)
 	(junction
+		(at 111.76 124.46)
+		(diameter 0)
+		(color 0 0 0 0)
+	)
+	(junction
 		(at 134.62 82.55)
 		(diameter 0)
@@
 	)
 	(junction
+		(at 118.11 111.76)
+		(diameter 0)
+		(color 0 0 0 0)
+	)
+	(junction
 		(at 186.69 87.63)
 		(diameter 0)
@@
 	(wire
 		(pts
+			(xy 105.41 120.65) (xy 105.41 124.46)
+		)
+		(stroke
+			(width 0)
+			(type default)
+		)
+	)
+	(wire
+		(pts
 			(xy 184.15 82.55) (xy 176.53 82.55)
 		)
@@
 	(wire
 		(pts
+			(xy 111.76 124.46) (xy 118.11 124.46)
+		)
+		(stroke
+			(width 0)
+			(type default)
+		)
+	)
+	(wire
+		(pts
 			(xy 20.32 54.61) (xy 20.32 50.8)
 		)
@@
 	(wire
 		(pts
-			(xy 118.11 121.92) (xy 118.11 127)
+			(xy 118.11 121.92) (xy 118.11 124.46)
+		)
+		(stroke
+			(width 0)
+			(type default)
+		)
+	)
+	(wire
+		(pts
+			(xy 105.41 111.76) (xy 118.11 111.76)
 		)
 		(stroke
@@
 	(wire
 		(pts
+			(xy 105.41 113.03) (xy 105.41 111.76)
+		)
+		(stroke
+			(width 0)
+			(type default)
+		)
+	)
+	(wire
+		(pts
 			(xy 27.94 50.8) (xy 27.94 54.61)
 		)
@@
 	(wire
 		(pts
+			(xy 111.76 124.46) (xy 111.76 127)
+		)
+		(stroke
+			(width 0)
+			(type default)
+		)
+	)
+	(wire
+		(pts
 			(xy 20.32 62.23) (xy 20.32 63.5)
 		)
@@
 	(wire
 		(pts
+			(xy 105.41 124.46) (xy 111.76 124.46)
+		)
+		(stroke
+			(width 0)
+			(type default)
+		)
+	)
+	(wire
+		(pts
 			(xy 24.13 50.8) (xy 27.94 50.8)
 		)
@@
 	(symbol
 		(lib_id "power:GNDREF")
-		(at 118.11 127 0)
+		(at 111.76 127 0)
 		(unit 1)
 		(exclude_from_sim no)
@@
 		(fields_autoplaced yes)
 		(property "Reference" "#PWR010"
-			(at 118.11 133.35 0)
+			(at 111.76 133.35 0)
 			(effects
 				(font
@@
 		)
 		(property "Value" "GNDREF"
-			(at 118.11 132.08 0)
+			(at 111.76 132.08 0)
 			(effects
 				(font
@@
 		)
 		(property "Footprint" ""
-			(at 118.11 127 0)
+			(at 111.76 127 0)
 			(effects
 				(font
@@
 		)
 		(property "Datasheet" ""
-			(at 118.11 127 0)
+			(at 111.76 127 0)
 			(effects
 				(font
@@
 		)
 		(property "Description" "Power symbol creates a global label with name \"GNDREF\" , reference supply ground"
-			(at 118.11 127 0)
+			(at 111.76 127 0)
 			(effects
 				(font
@@
 					(unit 1)
 				)
+			)
+		)
+	)
+	(symbol
+		(lib_id "Device:C")
+		(at 105.41 116.84 0)
+		(unit 1)
+		(exclude_from_sim no)
+		(in_bom yes)
+		(on_board yes)
+		(dnp no)
+		(fields_autoplaced yes)
+		(property "Reference" "C3"
+			(at 109.22 115.5699 0)
+			(effects
+				(font
+					(size 1.27 1.27)
+				)
+				(justify left)
+			)
+		)
+		(property "Value" "10nF"
+			(at 109.22 118.1099 0)
+			(effects
+				(font
+					(size 1.27 1.27)
+				)
+				(justify left)
+			)
+		)
+		(property "Footprint" "Capacitor_SMD:C_0603_1608Metric_Pad1.08x0.95mm_HandSolder"
+			(at 106.3752 120.65 0)
+			(effects
+				(font
+					(size 1.27 1.27)
+				)
+				(hide yes)
+			)
+		)
+		(property "Datasheet" "~"
+			(at 105.41 116.84 0)
+			(effects
+				(font
+					(size 1.27 1.27)
+				)
+				(hide yes)
+			)
+		)
+		(property "Description" "Unpolarized capacitor"
+			(at 105.41 116.84 0)
+			(effects
+				(font
+					(size 1.27 1.27)
+				)
+				(hide yes)
+			)
+		)
+		(pin "1"
+		)
+		(pin "2"
+		)
+		(instances
+			(project "temp_sensor"
+				(path "/b0b1ee9b-4b17-44f1-97bf-1e35f7090125"
+					(reference "C3")
+					(unit 1)
+				)
