File: temp_sensor.kicad_sch (KiCad schematic)
At the start: 27 parts, among them J2 Conn_01x06, J3 Conn_01x08, J4 Conn_01x08, SW1 Boot, SW2 Reset, U1 HDC3020DEFR, U2 ESP-12F, U3 TPS613221ADBVR, U4 TLV74033PDBVR

Commit message: Add old code and sch to then delete
Connections:
- net bust_vout: now reaches C4.1, JP2.1 (A), U4.5 (OUT)
- net MISO: now reaches J2.2 (Pin_2), R3.1, U2.10 (MISO)
- net boot: now reaches J4.4 (Pin_4), R5.1, SW1.2, U2.18 (GPIO0)
- net GPIO9: now reaches J2.3 (Pin_3), U2.11 (GPIO9)
- net GPIO10: now reaches J2.4 (Pin_4), U2.12 (GPIO10)
- net MOSI: now reaches J2.5 (Pin_5), U2.13 (MOSI)
- net SCLK: now reaches J2.6 (Pin_6), U2.14 (SCLK)
- net CS: now reaches J4.2 (Pin_2), R7.2, U2.16 (GPIO15)
- net led: now reaches J4.3 (Pin_3), U2.17 (GPIO2)
- net SDA: now reaches J4.5 (Pin_5), R1.1, U1.1 (SDA), U2.19 (GPIO4)
- net ADC: now reaches J3.2 (Pin_2), U2.2 (ADC)
- net SCL: now reaches J4.6 (Pin_6), R2.1, U1.4 (SCL), U2.20 (GPIO5)
- net rxd: now reaches J4.7 (Pin_7), U2.21 (GPIO3/RXD)
- net txd: now reaches J4.8 (Pin_8), U2.22 (GPIO1/TXD)
- net EN: now reaches J3.3 (Pin_3), R6.1, U2.3 (EN)
- net alert: now reaches J3.5 (Pin_5), U1.3 (ALERT), U2.5 (GPIO14)
- net GPIO12: now reaches J3.6 (Pin_6), U2.6 (GPIO12)
- net GPIO13: now reaches J3.7 (Pin_7), U2.7 (GPIO13)
- net CSO: now reaches J2.1 (Pin_1), U2.9 (CS0)
- net boost_vout: now reaches C2.1, JP1.1 (A), U3.4 (VOUT)
- net batt: now reaches C6.1, JP3.1 (A), L1.1, U4.1 (IN), U4.3 (EN), batt1.1 (+)
Other:
- moved on the sheet: R1, R2, R7
