File: temp_sensor.kicad_pcb (KiCad board)
At the start: 2 copper layers, 40 x 35 mm, 28 parts, among them J2 Conn_01x06, J3 Conn_01x08, J4 Conn_01x08, SW1 Boot, SW2 Reset, U1 HDC3020DEFR, U2 ESP-12F, U3 TPS613221ADBVR, U4 TLV74033PDBVR

Commit message: Add old code and sch to then delete
Connections:
- net Net-(J2-Pin_1) renamed /CSO
- net Net-(J2-Pin_2) renamed /MISO
- net Net-(J2-Pin_3) renamed /GPIO9
- net Net-(J2-Pin_4) renamed /GPIO10
- net Net-(J2-Pin_5) renamed /MOSI
- net Net-(J2-Pin_6) renamed /SCLK
- net Net-(J3-Pin_2) renamed /ADC
- net Net-(J3-Pin_3) renamed /EN
- net Net-(J3-Pin_5) renamed /alert
- net Net-(J3-Pin_6) renamed /GPIO12
- net Net-(J3-Pin_7) renamed /GPIO13
- net Net-(J4-Pin_2) renamed /CS
- net Net-(J4-Pin_3) renamed /led
- net Net-(J4-Pin_4) renamed /boot
- net Net-(J4-Pin_5) renamed /SDA
- net Net-(J4-Pin_6) renamed /SCL
- net Net-(J4-Pin_7) renamed /rxd
- net Net-(J4-Pin_8) renamed /txd
- net Net-(JP1-A) renamed /boost_vout
- net Net-(JP2-A) renamed /bust_vout
- net Net-(JP3-A) renamed /batt
